File: modulo_puente_h/modulo_puente_h.kicad_pcb (KiCad board)
At the start: 2 copper layers, 63 x 50 mm, 16 parts, among them J1 Conn_01x07_Pin, M1 Motor_IZQ, M2 Motor_DER, U1 L298N

Commit message: test commit
Routing:
- net /Entrada 1 Motor B: track 76.2 -> 79.0 mm
Changed lines of the file:
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@@
-	)
-	(segment
-		(start 93.615 46)
-		(end 63.5 46)
-		(width 0.7)
-		(layer "F.Cu")
-		(net 10)
-	)
-	(segment
-		(start 54 55.5)
-		(end 54 61)
-		(width 0.7)
-		(layer "F.Cu")
-		(net 10)
 	)
 	(segment
@@
 	)
 	(segment
+		(start 109 56.5)
+		(end 98.5 46)
+		(width 0.7)
+		(layer "F.Cu")
+		(net 10)
+	)
+	(segment
 		(start 63.5 46)
 		(end 54 55.5)
@@
 	)
 	(segment
-		(start 109 61.385)
-		(end 93.615 46)
+		(start 54 55.5)
+		(end 54 61)
 		(width 0.7)
 		(layer "F.Cu")
+		(net 10)
+	)
+	(segment
+		(start 98.5 46)
+		(end 63.5 46)
+		(width 0.7)
+		(layer "F.Cu")
+		(net 10)
+	)
+	(segment
+		(start 109 61.385)
+		(end 109 56.5)
+		(width 0.7)
+		(layer "F.Cu")
